File: board/hw-bms-48v.kicad_pcb (KiCad board)
At the start: 2 copper layers, 100 x 50 mm, 43 parts, among them J1 BATT, J3 CURRENT, J4 TEMP, J5 PROG, J6 ILI9225, U1 ESP32-C3-WROOM-02, U2 BD9G341EFJ, U3 LM1117MP-3.3

Commit message: WIP
Parts:
- moved J3 68.8 mm to (78.0, 64.2)
- moved J5 68.8 mm to (42.6, 97.4)
- moved J6 68.8 mm to (51.5, 61.6)
- moved RV1 68.8 mm to (61.9, 100.2)
- moved C1 68.8 mm to (56.2, 83.4)
- moved C2 68.8 mm to (56.2, 86.4)
- moved C3 68.8 mm to (56.2, 89.4)
- moved C4 68.8 mm to (56.2, 92.4)
- moved C5 68.8 mm to (56.2, 95.5)
- moved H1 68.8 mm to (44.7, 63.8)
- moved H2 68.8 mm to (44.7, 72.7)
- moved H3 68.8 mm to (44.7, 81.7)
- moved H4 68.8 mm to (44.7, 90.6)
- moved J4 68.8 mm to (86.5, 86.8)
- moved R1 68.8 mm to (70.6, 97.6)
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
Commit message: WIP
Parts:
- removed C13: 10u, Capacitor_SMD:C_0805_2012Metric_Pad1.18x1.45mm_HandSolder
- removed the C5 at (56.2, 95.5)
- removed the C7 at (61.0, 86.4)
- added C11: 47u, Capacitor_SMD:C_0805_2012Metric_Pad1.18x1.45mm_HandSolder, F.Cu at (126.0, 66.0)
- J2: renamed from J5; footprint Connector_PinHeader_2.54mm:PinHeader_1x03_P2.54mm_Vertical -> Connector_PinHeader_2.54mm:PinHeader_1x03_P2.54mm_Horizontal
- moved H3 147.2 mm to (190.0, 105.0)
- moved H2 145.5 mm to (190.0, 65.0)
- moved C6 137.6 mm to (193.0, 98.0), turned to 90 degrees
- moved C7 134.3 mm to (190.0, 98.0), turned to 90 degrees
- moved J2 133.0 mm to (175.5, 98.6), turned to -90 degrees
- moved C8 131.1 mm to (187.0, 98.0), turned to 90 degrees
- moved C12 127.5 mm to (188.0, 72.0)
- moved R12 119.4 mm to (192.0, 72.0), turned to 180 degrees
- moved R11 114.0 mm to (184.0, 98.0), turned to 90 degrees
- moved C10 90.9 mm to (147.0, 95.0)
- moved J5 86.4 mm to (130.0, 97.7), turned to 180 degrees
- moved RV1 83.5 mm to (144.9, 91.0), turned to 180 degrees
- moved J4 74.7 mm to (159.8, 101.2)
- moved R6 72.5 mm to (120.0, 76.0), turned to 180 degrees
- moved J3 72.1 mm to (140.0, 101.0)
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- renumbered C14 to C1, C4 to C10, C6 to C12, C9 to C2, C8 to C3, C10 to C4, C11 to C5, C1 to C6, C2 to C7, C3 to C8, C12 to C9, D2 to D1, D1 to D2, J6 to J5, R8 to R1, R4 to R10, R5 to R11, R6 to R12, R7 to R13, R9 to R2, R10 to R3, R11 to R4, R12 to R5, R13 to R6, R1 to R7, R2 to R8, R3 to R9, U2 to U1, U3 to U2, U1 to U3
Routing:
- net /LED: track 0.00 -> 101.8 mm, vias 0 -> 2
- net Net-(U3-GPIO0/ADC1_CH0/XTAL_32K_P): track 0.00 -> 94.3 mm, vias 0 -> 1
- net +5V: track 0.00 -> 73.9 mm
- net /LCD_SS: track 0.00 -> 72.8 mm, vias 0 -> 2
- net Net-(U3-GPIO1/ADC1_CH1/XTAL_32K_N): track 0.00 -> 64.4 mm, vias 0 -> 1
- net /LCD_BL: track 0.00 -> 63.3 mm, vias 0 -> 2
- net /LCD_SCK: track 0.00 -> 62.7 mm
- net /LCD_SDI: track 0.00 -> 60.3 mm
- net /LCD_RS: track 0.00 -> 57.9 mm
- net /LCD_RST: track 0.00 -> 56.7 mm, vias 0 -> 2
- net +BATT: track 0.00 -> 44.8 mm
- net Net-(J4-Pin_2): track 0.00 -> 32.7 mm
- net Net-(U1-FB): track 0.00 -> 27.4 mm, vias 0 -> 2
- net Net-(D1-K): track 0.00 -> 26.0 mm, vias 0 -> 2
- net +3V3: track 0.00 -> 25.1 mm, vias 0 -> 7
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- added copper zone on B.Cu, net +3V3
- added copper zone on F.Cu, net GND
Other:
- outline, holes or cut-outs redrawn
- board text added: "+"
- board text added: "-"
- board text added: "BMS-48V v1.0"
