File: board/hw-bms-48v.kicad_sch (KiCad schematic)
At the start: 24 parts, among them J1 BATT+, J1 BATT-, J2 PROG, J3 CURRENT, J4 TEMP, U2 BD9G341EFJ, U2 ESP32-C3-WROOM-02, U3 LM1117MP-3.3

Commit message: WIP
Parts:
- removed J1: BATT+, Connector_Wire:SolderWire-1sqmm_1x01_D1.4mm_OD3.9mm, symbol Connector_Generic:Conn_01x01
- removed J1: BATT-, Connector_Wire:SolderWire-1sqmm_1x01_D1.4mm_OD3.9mm, symbol Connector_Generic:Conn_01x01
- removed J2: PROG, Connector_PinHeader_2.54mm:PinHeader_1x03_P2.54mm_Vertical, symbol Connector:Conn_01x03_Female
- added C10: ???, Capacitor_SMD:C_0805_2012Metric_Pad1.18x1.45mm_HandSolder, symbol Device:C
- added C11, C12: 47u, Capacitor_SMD:C_0805_2012Metric_Pad1.18x1.45mm_HandSolder, symbol Device:C
- added C13: 10u, Capacitor_SMD:C_0805_2012Metric_Pad1.18x1.45mm_HandSolder, symbol Device:C
- added C14: 10u/100V, Capacitor_SMD:C_0805_2012Metric_Pad1.18x1.45mm_HandSolder, symbol Device:C
- added C8: 100n, Capacitor_SMD:C_0805_2012Metric_Pad1.18x1.45mm_HandSolder, symbol Device:C
- added C9: 6n8, Capacitor_SMD:C_0805_2012Metric_Pad1.18x1.45mm_HandSolder, symbol Device:C
- added D1: SK22, Diode_SMD:D_SMB, symbol Device:D_Schottky
- added H1, H2, H3, H4: MountingHole, MountingHole:MountingHole_3.7mm_Pad_Via, symbol Mechanical:MountingHole
- added J1: BATT, Drake:DG235-3.81-02P, symbol Connector_Generic:Conn_01x02
- added J5: PROG, Connector_PinHeader_2.54mm:PinHeader_1x03_P2.54mm_Vertical, symbol Connector_Generic:Conn_01x03
- added J6: ILI9225, Connector_PinSocket_2.54mm:PinSocket_1x11_P2.54mm_Vertical, symbol Connector_Generic:Conn_01x11
- added L3: 33uH, Inductor_SMD:L_12x12mm_H6mm, symbol Device:L
- added R10: 47k, Resistor_SMD:R_0805_2012Metric_Pad1.20x1.40mm_HandSolder, symbol Device:R
- added R11: 10k, Resistor_SMD:R_0805_2012Metric_Pad1.20x1.40mm_HandSolder, symbol Device:R
- added R12: 3k, Resistor_SMD:R_0805_2012Metric_Pad1.20x1.40mm_HandSolder, symbol Device:R
- added R13: 750R, Resistor_SMD:R_0805_2012Metric_Pad1.20x1.40mm_HandSolder, symbol Device:R
- added R8: 100k, Resistor_SMD:R_0805_2012Metric_Pad1.20x1.40mm_HandSolder, symbol Device:R
- added R9: 20k, Resistor_SMD:R_0805_2012Metric_Pad1.20x1.40mm_HandSolder, symbol Device:R
Connections:
- net +3V3: now also U3.2 (VO), C13.2
- net +5V: now also U3.3 (VI), C11.2, C12.2, J6.1 (Pin_1), L3.2, R12.1
- net +BATT: now also U2.8 (VCC), C14.2, J1.2 (Pin_2), R8.1
- net GND: now also U2.2 (GND), U3.1 (GND), C10.1, C11.1, C12.1, C13.1, C14.1, D1.2 (A), J1.1 (Pin_1), J5.2 (Pin_2), J6.2 (Pin_2), J6.3 (Pin_3), R10.2, R11.2, R13.2, R9.2
- net USB_D+: now also J5.1 (Pin_1)
- net USB_D-: now also J5.3 (Pin_3)
- net LCD_SS: now reaches U2.10 (GPIO10)
- net LCD_SS: now also J6.11 (Pin_11)
- net LCD_BL: now reaches U2.11 (GPIO20/U0RXD)
- net LCD_BL: now also J6.6 (Pin_6)
- net LCD_SCK: now reaches U2.5 (GPIO6)
- net LCD_SCK: now also J6.7 (Pin_7)
- net LCD_SDI: now reaches U2.6 (GPIO7)
- net LCD_SDI: now also J6.8 (Pin_8)
- net LCD_RS: now reaches U2.7 (GPIO8)
- net LCD_RS: now also J6.9 (Pin_9)
- net LCD_RST: now reaches U2.8 (GPIO9)
- net LCD_RST: now also J6.10 (Pin_10)
- net at U2.1 (LX): now also C8.1, D1.1 (K), L3.1
- net at U2.3 (VC): now also C10.2, C9.2
- net at U2.4 (FB): now also R12.2, R13.1
- net at U2.5 (RT): now also R10.1
- net at U2.6 (EN): now also R8.2, R9.1
- net at U2.7 (BST): now also C8.2
- new net: C9.1, R11.1
- no-connect marks 9 -> 5
Other:
- note removed: "pridat zdroj 3v3 5v displej"
- moved on the sheet: C1, C2, C3, C4, C5, C6, C7, D1, J3, J4, R1, R2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

Commit message: WIP
Parts:
- removed C13: 10u, Capacitor_SMD:C_0805_2012Metric_Pad1.18x1.45mm_HandSolder, symbol Device:C
- removed C5, C7: 47u, Capacitor_SMD:C_0805_2012Metric_Pad1.18x1.45mm_HandSolder, symbol Device:C
- added C11: 47u, Capacitor_SMD:C_0805_2012Metric_Pad1.18x1.45mm_HandSolder, symbol Device:C
- J2: renamed from J5; footprint Connector_PinHeader_2.54mm:PinHeader_1x03_P2.54mm_Vertical -> Connector_PinHeader_2.54mm:PinHeader_1x03_P2.54mm_Horizontal
- R5: renamed from R12; value 3k -> 3k (3.9k?)
- renumbered C14 to C1, C4 to C10, C6 to C12, C9 to C2, C8 to C3, C10 to C4, C11 to C5, C1 to C6, C2 to C7, C3 to C8, C12 to C9, J6 to J5, R8 to R1, R4 to R10, R5 to R11, R6 to R12, R9 to R2, R10 to R3, R11 to R4, R13 to R6, R1 to R7, R2 to R8, R3 to R9, U2 to U1, U3 to U2
Connections:
- net +3V3: now also C11.2
- net GND: now also C11.1
Other:
- note added: "The IC seems to be regulating to 840mV instead of expected 1V. 5V is then acheived by changing R5 to 3.9k."
- note added: "next version fixes: - C1 - replace by 4pcs 10uF/50V 1206 - Horizontal trimmer"

Commit message: WIP
Other:
- note added: "next version fixes: - C1 - replace by 4pcs 10uF/50V 1206 - Horizontal trimmer - FIX GROUND LOOPS (USB.GND->ESP32.GND)"
- note removed: "next version fixes: - C1 - replace by 4pcs 10uF/50V 1206 - Horizontal trimmer"
Changed lines of the file:
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@@
     (stroke (width 0) (type default))
   )
-  (text "next version fixes:\n- C1 - replace by 4pcs 10uF/50V 1206\n- Horizontal trimmer" (exclude_from_sim no)
+  (text "next version fixes:\n- C1 - replace by 4pcs 10uF/50V 1206\n- Horizontal trimmer\n- FIX GROUND LOOPS (USB.GND->ESP32.GND)" (exclude_from_sim no)
     (at 26.67 109.22 0)
     (effects (font (size 1.27 1.27)) (justify left bottom))

Commit message: WIP
Other:
- note added: "next version fixes: - C1 - replace by 4pcs 10uF/50V 1206 - Horizontal trimmer - FIX GROUND LOOPS (USB.GND->ESP32.GND) - ADC by PCF8591?"
- note removed: "next version fixes: - C1 - replace by 4pcs 10uF/50V 1206 - Horizontal trimmer - FIX GROUND LOOPS (USB.GND->ESP32.GND)"
Changed lines of the file:
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@@
     (stroke (width 0) (type default))
   )
-  (text "next version fixes:\n- C1 - replace by 4pcs 10uF/50V 1206\n- Horizontal trimmer\n- FIX GROUND LOOPS (USB.GND->ESP32.GND)" (exclude_from_sim no)
+  (text "next version fixes:\n- C1 - replace by 4pcs 10uF/50V 1206\n- Horizontal trimmer\n- FIX GROUND LOOPS (USB.GND->ESP32.GND)\n- ADC by PCF8591?" (exclude_from_sim no)
     (at 26.67 109.22 0)
     (effects (font (size 1.27 1.27)) (justify left bottom))
